File: satOBCs.kicad_pcb (KiCad board)
At the start: 2 copper layers, 55 x 94.5 mm, 10 parts, among them J1 Battery power, J2 sensor, U1 BMP280, U2 mpu-9250, U3 AZ1117-3.3, U6 DHT11

Commit message: 3rd time commit
Parts:
- removed LoRa_Ra-02_SX1278_433MHz2: ~, prashantkicadlibrary:LORA-02
- removed U1: BMP280, Package_LGA:Bosch_LGA-8_2x2.5mm_P0.65mm_ClockwisePinNumbering
- removed the U3 at (142.2, 115.2)
- removed the U3 at (210.5, 89.0)
- added D1: LED, LED_THT:LED_D4.0mm, F.Cu at (158.7, 54.0)
- added J3: Conn_01x10_Pin, Connector_PinHeader_2.54mm:PinHeader_1x10_P2.54mm_Vertical, F.Cu at (140.5, 107.8)
- added R1: R, Resistor_THT:R_Axial_DIN0207_L6.3mm_D2.5mm_P7.62mm_Horizontal, F.Cu at (145.7, 54.0)
- added SW1: SW_Push, Button_Switch_THT:SW_PUSH_6mm, F.Cu at (113.7, 121.8)
- added U3: AZ1117-3.3, Package_TO_SOT_SMD:SOT-89-3_Handsoldering, B.Cu at (149.0, 75.5)
- J2: value sensor -> Conn_01x10_Pin; footprint Connector_PinSocket_2.54mm:PinSocket_1x04_P2.54mm_Vertical -> Connector_PinHeader_2.54mm:PinHeader_1x10_P2.54mm_Vertical
- R2: value 10K -> R; footprint Resistor_SMD:R_0603_1608Metric -> Resistor_THT:R_Axial_DIN0207_L6.3mm_D2.5mm_P7.62mm_Horizontal
- moved U6 88.8 mm to (127.2, 120.1), turned to 90 degrees
- moved NodeMCU_v1 64.4 mm to (135.4, 71.2)
- moved U2 64.4 mm to (130.7, 70.0)
- moved J1 64.4 mm to (157.0, 77.0)
- moved J2 47.1 mm to (140.5, 55.0)
- moved R2 40.6 mm to (122.3, 122.2), turned to 90 degrees
Connections:
- J2 pad 1: GND -> /CS
- J2 pad 2: +3V3 -> /MOSI
- J2 pad 3: /SDA -> /MISO
- J2 pad 4: /SCL -> /SCLK
Routing:
- net +3V3: track 28.0 -> 95.5 mm
- net /RST: track 0.00 -> 22.5 mm
- net /DHT_data: track 0.00 -> 17.9 mm
- net /CS: track 0.00 -> 6.26 mm
- net /MISO: track 0.00 -> 5.80 mm
- net /SCLK: track 0.00 -> 5.78 mm
- net /MOSI: track 0.00 -> 5.78 mm
- net /VIN: track 0.00 -> 5.55 mm
- net /SCL: track 16.4 -> 20.6 mm
- net /SDA: track 16.4 -> 20.4 mm
- net Net-(D1-A): track 0.00 -> 2.83 mm
- added copper zone on B.Cu, net GND
- added copper zone on F.Cu, net GND
Other:
- board size 55 x 94.5 mm -> 55.2 x 94.2 mm

Commit message: 4th edited
Parts:
- J3: moved to B.Cu
- moved J3 26.3 mm to (136.6, 133.8), turned to 90 degrees
- moved R2 12.0 mm to (113.6, 130.5)
- moved U6 7.47 mm to (121.5, 124.9)
- moved SW1 6.50 mm to (113.8, 115.3), turned to 0 degrees
- moved D1 5.17 mm to (153.7, 52.7)
- moved R1 5.17 mm to (140.7, 52.7)
- moved U2 5.10 mm to (126.1, 67.8)
- moved J1 5.10 mm to (152.4, 74.8)
- moved J2 5.10 mm to (135.9, 52.8)
- moved NodeMCU_v1 5.10 mm to (130.8, 69.0)
- moved U3 5.10 mm to (144.4, 73.3)
Routing:
- net /RST: track 22.5 -> 4.00 mm
- net +3V3: track 95.5 -> 79.2 mm
- net /DHT_data: track 17.9 -> 4.77 mm
Other:
- board size 55.2 x 94.2 mm -> 51 x 90.4 mm

Commit message: added last
Parts:
- removed J3: Conn_01x10_Pin, Connector_PinHeader_2.54mm:PinHeader_1x10_P2.54mm_Vertical
- added J4: Conn_01x11_Pin, Connector_PinSocket_2.54mm:PinSocket_1x11_P2.54mm_Vertical, B.Cu at (139.5, 58.0)
- added LoRa_Ra-02_SX1278_433MHz1: ~, prashantkicadlibrary:LORA-02, F.Cu at (154.4, 107.9)
- added U1: BMP280, Connector_PinHeader_2.54mm:PinHeader_1x06_P2.54mm_Vertical, B.Cu at (131.3, 116.5)
- J2: value Conn_01x10_Pin -> Conn_01x11_Pin; footprint Connector_PinHeader_2.54mm:PinHeader_1x10_P2.54mm_Vertical -> Connector_PinSocket_2.54mm:PinSocket_1x11_P2.54mm_Vertical
- moved J2 73.4 mm to (138.2, 126.2)
- moved R1 14.7 mm to (142.8, 67.2)
- moved SW1 12.4 mm to (115.0, 103.0), turned to -90 degrees
- moved R2 7.76 mm to (112.7, 122.8)
- moved D1 6.64 mm to (149.8, 58.1), turned to 0 degrees
- moved J1 5.32 mm to (153.5, 80.0)
- moved NodeMCU_v1 5.32 mm to (131.9, 74.2)
- moved U2 5.32 mm to (127.2, 73.0)
- moved U3 5.32 mm to (145.5, 78.5)
- moved U6 5.19 mm to (118.9, 120.4)
Connections:
- J2 pad 10: /RST -> /SCL
- J2 pad 6: /DHT_data -> /D3
- J2 pad 7: +3V3 -> /DHT_data
- J2 pad 8: /SDA -> +3V3
- J2 pad 9: /SCL -> /SDA
- NodeMCU_v1 pad 26: /DHT_data -> /D3
- NodeMCU_v1 pad 27: /D3 -> /DHT_data
- R1 pad 1: /LED -> +3V3
Routing:
- net +3V3: track 79.2 -> 162.1 mm
- net /RST: track 4.00 -> 67.7 mm
- net /D3: track 0.00 -> 48.9 mm, vias 0 -> 2
- net /SDA: track 20.4 -> 51.4 mm, vias 0 -> 2
- net /SCL: track 20.6 -> 46.4 mm, vias 0 -> 2
- net /MISO: track 5.80 -> 23.4 mm
- net /SCLK: track 5.78 -> 21.7 mm, vias 0 -> 2
- net /MOSI: track 5.78 -> 20.6 mm
- net /CS: track 6.26 -> 15.1 mm
- net /DHT_data: track 4.77 -> 12.2 mm
- net Net-(D1-A): track 2.83 -> 10.0 mm
Other:
- board size 51 x 90.4 mm -> 51.1 x 77.5 mm
