File: satOBCs.kicad_sch (KiCad schematic)
At the start: 12 parts, among them J1 Battery power, J2 temperature sensor, J3 temperature sensor, J6 pulse/oxygen sensor, U1 ESP32-WROOM-32E-N8R2, U2 mpu-9250, U3 AZ1117-3.3, U4 DHT11, U5 BMP280

Commit message: added 2
Parts:
- removed J3: temperature sensor, Connector_PinSocket_2.54mm:PinSocket_1x04_P2.54mm_Vertical, symbol Connector:Conn_01x04_Pin
- removed J6: pulse/oxygen sensor, Connector_PinSocket_2.54mm:PinSocket_1x04_P2.54mm_Vertical, symbol Connector:Conn_01x04_Pin
- removed LoRa_Ra-02_SX1278_433MHz1: ~, symbol Cube_Sat:lora
- removed R3: 10K, Resistor_THT:R_Axial_DIN0207_L6.3mm_D2.5mm_P7.62mm_Horizontal, symbol Device:R
- removed U1: ESP32-WROOM-32E-N8R2, prashantkicadlibrary:MODULE_ESP32_DEVKIT_V1, symbol symbols:ESP32-WROOM-32_DEV_BOARD
- removed U4: DHT11, Sensor:Aosong_DHT11_5.5x12.0_P2.54mm, symbol Sensor:DHT11
- removed U5: BMP280, Package_LGA:Bosch_LGA-8_2x2.5mm_P0.65mm_ClockwisePinNumbering, symbol Cube_Sat:BMP280
- added D1: LED, LED_THT:LED_D4.0mm, symbol Device:LED
- added LoRa_Ra-02_SX1278_433MHz2: ~, prashantkicadlibrary:LORA-02, symbol Cube_Sat:lora
- added NodeMCU_v1: ~, prashantkicadlibrary:nodemcu, symbol Cube_Sat:node_mcu
- added R1: R, Resistor_THT:R_Axial_DIN0207_L6.3mm_D2.5mm_P7.62mm_Horizontal, symbol Device:R
- added SW1: SW_Push, easyeda2kicad:SW-SMD_L6.0-W3.3-LS8.0, symbol Switch:SW_Push
- added U1: BMP280, Package_LGA:Bosch_LGA-8_2x2.5mm_P0.65mm_ClockwisePinNumbering, symbol Cube_Sat:BMP280
- added U6: DHT11, Sensor:Aosong_DHT11_5.5x12.0_P2.54mm, symbol Sensor:DHT11
- J2: value temperature sensor -> sensor
- R2: value 10K -> R
- U3: footprint (none) -> Package_TO_SOT_SMD:SOT-89-3_Handsoldering
Connections:
- net +3V3: now also LoRa_Ra-02_SX1278_433MHz2.5 (3.3V), NodeMCU_v1.11 (3V), U1.1 (VCC), U1.5 (CSB), U6.1 (VDD)
- net GND: now also D1.1 (K), LoRa_Ra-02_SX1278_433MHz2.3 (GND), NodeMCU_v1.14 (G), SW1.1, U1.2 (GND), U1.6 (SDO), U6.4 (GND)
- net IO21 renamed SDA
- net SDA: now also NodeMCU_v1.28 (D2), U1.4 (SDA)
- net IO22 renamed SCL
- net SCL: now also NodeMCU_v1.29 (D1), U1.3 (SCL)
- net SW2 renamed RST
- net RST: now also LoRa_Ra-02_SX1278_433MHz2.7 (DIO3), NodeMCU_v1.30 (D0), SW1.2
- new net: D1.2 (A), R1.2
- new net: NodeMCU_v1.15 (GND), NodeMCU_v1.38 (GND), NodeMCU_v1.39 (GND)
- new net: NodeMCU_v1.19 (RX), NodeMCU_v1.20 (D8), NodeMCU_v1.32 (NC)
- new net CS: LoRa_Ra-02_SX1278_433MHz2.4 (NSS), NodeMCU_v1.20 (D8)
- new net D3: LoRa_Ra-02_SX1278_433MHz2.7 (DIO3), NodeMCU_v1.27 (D3)
- new net DHT_data: NodeMCU_v1.26 (D4), U6.2 (DATA)
- new net LED: R1.1
- new net MISO: LoRa_Ra-02_SX1278_433MHz2.8 (GND), NodeMCU_v1.22 (D6)
- new net MOSI: LoRa_Ra-02_SX1278_433MHz2.6 (MOSI), NodeMCU_v1.21 (D7)
- new net SCLK: LoRa_Ra-02_SX1278_433MHz2.8 (GND), NodeMCU_v1.23 (D5)
- no-connect marks 26 -> 33
Other:
- note added: "LED"
- note added: "MPU-9250 / MPU -6500"
- note added: "Micro Controller Node"
- note added: "SIGNAL BUTTONS"
- note removed: "Fall Detection Sensor MPU-9250 / MPU -6500"
- note removed: "Micro Controller (Esp32 Dev Modulle)"
- note removed: "Pins For Temperature Sensor"
- note removed: "Sensor"
- moved on the sheet: J1, J2, U2, U3

Commit message: 3rd time commit
Parts:
- removed J2: sensor, Connector_PinSocket_2.54mm:PinSocket_1x04_P2.54mm_Vertical, symbol Connector:Conn_01x04_Pin
- added J2, J3: Conn_01x10_Pin, Connector_PinHeader_2.54mm:PinHeader_1x10_P2.54mm_Vertical, symbol Connector:Conn_01x10_Pin
- SW1: footprint easyeda2kicad:SW-SMD_L6.0-W3.3-LS8.0 -> Button_Switch_THT:SW_PUSH_6mm
Connections:
- net +3V3: now also J2.7 (Pin_7), J3.7 (Pin_7)
- net CS: now also J2.1 (Pin_1), J3.1 (Pin_1)
- net DHT_data: now also J2.6 (Pin_6), J3.6 (Pin_6)
- net GND: now also J2.5 (Pin_5), J3.5 (Pin_5)
- net MISO: now also J2.3 (Pin_3), J3.3 (Pin_3)
- net MOSI: now also J2.2 (Pin_2), J3.2 (Pin_2)
- net RST: now also J2.10 (Pin_10), J3.10 (Pin_10)
- net SCL: now also J2.9 (Pin_9), J3.9 (Pin_9)
- net SCLK: now also J2.4 (Pin_4), J3.4 (Pin_4)
- net SDA: now also J2.8 (Pin_8), J3.8 (Pin_8)
- net at NodeMCU_v1.15 (GND): now also NodeMCU_v1.38 (GND), NodeMCU_v1.39 (GND)
- net at NodeMCU_v1.19 (RX): now also NodeMCU_v1.20 (D8), NodeMCU_v1.32 (NC)

Commit message: added last
Parts:
- removed J2, J3: Conn_01x10_Pin, Connector_PinHeader_2.54mm:PinHeader_1x10_P2.54mm_Vertical, symbol Connector:Conn_01x10_Pin
- removed LoRa_Ra-02_SX1278_433MHz2: ~, prashantkicadlibrary:LORA-02, symbol Cube_Sat:lora
- added J2, J4: Conn_01x11_Pin, Connector_PinSocket_2.54mm:PinSocket_1x11_P2.54mm_Vertical, symbol Connector:Conn_01x11_Pin
- added LoRa_Ra-02_SX1278_433MHz1: ~, prashantkicadlibrary:LORA-02, symbol prashantkicadlibrary:lora
- U1: footprint Package_LGA:Bosch_LGA-8_2x2.5mm_P0.65mm_ClockwisePinNumbering -> Connector_PinHeader_2.54mm:PinHeader_1x06_P2.54mm_Vertical
Connections:
- net LED is gone; now on net +3V3: R1.1
- net +3V3: now also J2.8 (Pin_8), J4.8 (Pin_8), LoRa_Ra-02_SX1278_433MHz1.5 (3.3V)
- net CS: now also J2.1 (Pin_1), J4.1 (Pin_1), LoRa_Ra-02_SX1278_433MHz1.4 (NSS)
- net D3: now also NodeMCU_v1.26 (D4), J2.6 (Pin_6), J4.6 (Pin_6), LoRa_Ra-02_SX1278_433MHz1.9 (DIO0); no longer NodeMCU_v1.27 (D3)
- net DHT_data: now also NodeMCU_v1.27 (D3), J2.7 (Pin_7), J4.7 (Pin_7); no longer NodeMCU_v1.26 (D4)
- net GND: now also J2.5 (Pin_5), J4.5 (Pin_5), LoRa_Ra-02_SX1278_433MHz1.3 (GND)
- net MISO: now also J2.3 (Pin_3), J4.3 (Pin_3), LoRa_Ra-02_SX1278_433MHz1.8 (MISO)
- net MOSI: now also J2.2 (Pin_2), J4.2 (Pin_2), LoRa_Ra-02_SX1278_433MHz1.6 (MOSI)
- net RST: now also J2.11 (Pin_11), J4.11 (Pin_11), LoRa_Ra-02_SX1278_433MHz1.7 (RST)
- net SCL: now also J2.10 (Pin_10), J4.10 (Pin_10)
- net SCLK: now also J2.4 (Pin_4), J4.4 (Pin_4), LoRa_Ra-02_SX1278_433MHz1.10 (SCK)
- net SDA: now also J2.9 (Pin_9), J4.9 (Pin_9)
- net at NodeMCU_v1.15 (GND): now also NodeMCU_v1.38 (GND), NodeMCU_v1.39 (GND)
- net at NodeMCU_v1.19 (RX): now also NodeMCU_v1.20 (D8), NodeMCU_v1.32 (NC)
Other:
- note added: "BMP280 , Pressure Sensor"
- note added: "DHT11 , Temperature Sensor"
- note added: "Device Reset Button"
- note added: "Headers Pin , Pcb 1 Master"
- note added: "Headers Pin, Pcb 2"
- note added: "Lora Moudle, Communication"
- note removed: "SIGNAL BUTTONS"
- moved on the sheet: D1, J1, NodeMCU_v1, R1, R2, SW1, U1, U2, U3, U6
